Commit message: bot spawned and situps done

File: go2_description/xacro/robot.xacro (robot description, xacro)
@@ -11,5 +11,5 @@
     <!-- find-pkg-share -->
     <!-- <xacro:include filename="$(find go2_description)/xacro/stairs.xacro"/> -->
-    <!-- <xacro:include filename="$(find go2_description)/xacro/gazebo.xacro"/> -->
+    <xacro:include filename="$(find go2_description)/xacro/gazebo.xacro"/>
     <!-- <xacro:include filename="$(find go2_gazebo)/launch/stairs.urdf.xacro"/> -->
     <!-- <xacro:stairs stairs="15" xpos="0" ypos="0" zpos="0" /> -->
@@ -19,10 +19,10 @@
     <!-- <xacro:if value="$(arg DEBUG)">
     </xacro:if>  -->
-    <link name="world"/>
+    <!-- <link name="world"/>
     <joint name="base_static_joint" type="fixed">
         <origin rpy="0 0 0" xyz="0 0 0"/>
         <parent link="world"/>
         <child link="base"/>
-    </joint>
+    </joint> -->
     <link name="base">
         <visual>
