Commit message: go2 goes to goal in aws warehouse

File: go2_description/xacro/const.xacro (robot description, xacro)
@@ -39,64 +39,92 @@
     <xacro:property name="calf_offset_z" value="-0.213"/>
     <!-- joint limits -->
-    <xacro:property name="damping" value="0.0"/>
-    <xacro:property name="friction" value="0.0"/>
+    <xacro:property name="damping" value="0.5"/>
+    <xacro:property name="friction" value="0.5"/>
     <xacro:property name="hip_position_max" value="1.0472"/>
     <xacro:property name="hip_position_min" value="-1.0472"/>
-    <xacro:property name="hip_velocity_max" value="30.1"/>
+    <xacro:property name="hip_velocity_max" value="1.5"/>
+    <!-- <xacro:property name="hip_velocity_max" value="30.1"/> -->
     <xacro:property name="hip_torque_max" value="23.7"/>
     <xacro:property name="thigh_position_max" value="3.4907"/>
     <xacro:property name="thigh_position_min" value="-1.5708"/>
-    <xacro:property name="thigh_velocity_max" value="30.1"/>
+    <xacro:property name="thigh_velocity_max" value="1.5"/>
+    <!-- <xacro:property name="thigh_velocity_max" value="30.1"/> -->
     <xacro:property name="thigh_torque_max" value="23.7"/>
     <xacro:property name="calf_position_max" value="-0.83776"/>
     <xacro:property name="calf_position_min" value="-2.7227"/>
-    <xacro:property name="calf_velocity_max" value="20.06"/>
-    <xacro:property name="calf_torque_max" value="35.55"/>
+    <xacro:property name="calf_velocity_max" value="1.5"/>
+    <!-- <xacro:property name="calf_velocity_max" value="20.06"/> -->
+    <!-- <xacro:property name="calf_torque_max" value="35.55"/> -->
+    <xacro:property name="calf_torque_max" value="25"/>
     <!-- dynamics inertial value -->
     <!-- trunk -->
     <xacro:property name="trunk_mass" value="6.921"/>
+    <!-- <xacro:property name="trunk_mass" value="6.921"/> -->
+    <!-- <xacro:property name="trunk_mass" value="2"/> -->
     <xacro:property name="trunk_com_x" value="0.021112"/>
     <xacro:property name="trunk_com_y" value="0.00"/>
     <xacro:property name="trunk_com_z" value="-0.005366"/>
-    <xacro:property name="trunk_ixx" value="0.02448"/>
+    <xacro:property name="trunk_ixx" value="0.01683"/>
+    <xacro:property name="trunk_ixy" value="0.0"/>
+    <xacro:property name="trunk_ixz" value="0.0"/>
+    <xacro:property name="trunk_iyy" value="0.044483"/>
+    <xacro:property name="trunk_iyz" value="0"/>
+    <xacro:property name="trunk_izz" value="0.055683"/>
+    <!-- <xacro:property name="trunk_ixx" value="0.02448"/>
     <xacro:property name="trunk_ixy" value="0.00012166"/>
     <xacro:property name="trunk_ixz" value="0.0014849"/>
     <xacro:property name="trunk_iyy" value="0.098077"/>
     <xacro:property name="trunk_iyz" value="-3.12E-05"/>
-    <xacro:property name="trunk_izz" value="0.107"/>
+    <xacro:property name="trunk_izz" value="0.107"/> -->
     <!-- hip (left front) -->
     <xacro:property name="hip_mass" value="0.678"/>
+    <!-- <xacro:property name="hip_mass" value="0.250"/> -->
     <xacro:property name="hip_com_x" value="-0.0054"/>
     <xacro:property name="hip_com_y" value="0.00194"/>
     <xacro:property name="hip_com_z" value="-0.000105"/>
     <xacro:property name="hip_ixx" value="0.00048"/>
-    <xacro:property name="hip_ixy" value="-3.01E-06"/>
-    <xacro:property name="hip_ixz" value="1.11E-06"/>
+    <xacro:property name="hip_ixy" value="0.0"/>
+    <!-- <xacro:property name="hip_ixy" value="-3.01E-06"/> -->
+    <xacro:property name="hip_ixz" value="0.0"/>
+    <!-- <xacro:property name="hip_ixz" value="1.11E-06"/> -->
     <xacro:property name="hip_iyy" value="0.000884"/>
-    <xacro:property name="hip_iyz" value="-1.42E-06"/>
+    <xacro:property name="hip_iyz" value="0.0"/>
+    <!-- <xacro:property name="hip_iyz" value="-1.42E-06"/> -->
     <xacro:property name="hip_izz" value="0.000596"/>
     <!-- thigh -->
-    <xacro:property name="thigh_mass" value="1.152"/>
+    <!-- <xacro:property name="thigh_mass" value="1.152"/> -->
+    <xacro:property name="thigh_mass" value="0.552"/>
+    <!-- <xacro:property name="thigh_mass" value="0.125"/> -->
     <xacro:property name="thigh_com_x" value="-0.00374"/>
     <xacro:property name="thigh_com_y" value="-0.0223"/>
     <xacro:property name="thigh_com_z" value="-0.0327"/>
     <xacro:property name="thigh_ixx" value="0.00584"/>
-    <xacro:property name="thigh_ixy" value="8.72E-05"/>
-    <xacro:property name="thigh_ixz" value="-0.000289"/>
-    <xacro:property name="thigh_iyy" value="0.0058"/>
-    <xacro:property name="thigh_iyz" value="0.000808"/>
-    <xacro:property name="thigh_izz" value="0.00103"/>
+    <!-- <xacro:property name="thigh_ixx" value="0.00584"/> -->
+    <xacro:property name="thigh_ixy" value="0.0"/>
+    <!-- <xacro:property name="thigh_ixy" value="8.72E-05"/> -->
+    <xacro:property name="thigh_ixz" value="-0.0"/>
+    <!-- <xacro:property name="thigh_ixz" value="-0.000289"/> -->
+    <xacro:property name="thigh_iyy" value="0.0011"/>
+    <!-- <xacro:property name="thigh_iyy" value="0.0058"/> -->
+    <xacro:property name="thigh_iyz" value="0.0"/>
+    <!-- <xacro:property name="thigh_iyz" value="0.000808"/> -->
+    <xacro:property name="thigh_izz" value="3.29E-05"/>
+    <!-- <xacro:property name="thigh_izz" value="0.00103"/> -->
     <!-- calf -->
-    <xacro:property name="calf_mass" value="0.154"/>
+    <!-- <xacro:property name="calf_mass" value="0.154"/> -->
+    <xacro:property name="calf_mass" value="0.125"/>
     <xacro:property name="calf_com_x" value="0.00548"/>
     <xacro:property name="calf_com_y" value="-0.000975"/>
     <xacro:property name="calf_com_z" value="-0.115"/>
     <xacro:property name="calf_ixx" value="0.00108"/>
-    <xacro:property name="calf_ixy" value="3.4E-07"/>
-    <xacro:property name="calf_ixz" value="1.72E-05"/>
+    <xacro:property name="calf_ixy" value="0"/>
+    <!-- <xacro:property name="calf_ixy" value="3.4E-07"/> -->
+    <xacro:property name="calf_ixz" value="0"/>
+    <!-- <xacro:property name="calf_ixz" value="1.72E-05"/> -->
     <xacro:property name="calf_iyy" value="0.0011"/>
-    <xacro:property name="calf_iyz" value="8.28E-06"/>
+    <xacro:property name="calf_iyz" value="0"/>
+    <!-- <xacro:property name="calf_iyz" value="8.28E-06"/> -->
     <xacro:property name="calf_izz" value="3.29E-05"/>
     <!-- foot -->
-    <xacro:property name="foot_mass" value="0.06"/>
+    <xacro:property name="foot_mass" value="0.006"/>
 </robot>

File: go2_description/xacro/go2_leg.xacro (robot description, xacro)
@@ -17,5 +17,5 @@
             </xacro:if>
             <parent link="trunk"/>
-            <child link="${name}_hip"/>
+            <child link="${name}_hip_link"/>
             <axis xyz="1 0 0"/>
             <dynamics damping="${damping}" friction="${friction}"/>
@@ -27,5 +27,5 @@
             </xacro:if>
         </joint>
-        <link name="${name}_hip">
+        <link name="${name}_hip_link">
             <visual>
                 <xacro:if value="${(mirror_dae == True) and (front_hind_dae == True)}">
@@ -64,13 +64,13 @@
             </inertial>
         </link>
-        <joint name="${name}_thigh_joint" type="revolute">
+        <joint name="${name}_upper_leg_joint" type="revolute">
             <origin rpy="0 0 0" xyz="0 ${thigh_offset*mirror} 0"/>
-            <parent link="${name}_hip"/>
-            <child link="${name}_thigh"/>
+            <parent link="${name}_hip_link"/>
+            <child link="${name}_upper_leg_link"/>
             <axis xyz="0 1 0"/>
             <dynamics damping="${damping}" friction="${friction}"/>
             <limit effort="${thigh_torque_max}" velocity="${thigh_velocity_max}" lower="${thigh_position_min}" upper="${thigh_position_max}"/>
         </joint>
-        <link name="${name}_thigh">
+        <link name="${name}_upper_leg_link">
             <visual>
                 <origin rpy="0 0 0" xyz="0 0 0"/>
@@ -93,5 +93,11 @@
             <inertial>
                 <origin rpy="0 0 0" xyz="${thigh_com_x} ${thigh_com_y*mirror} ${thigh_com_z}"/>
-                <mass value="${thigh_mass}"/>
+                <xacro:if value="${front_hind == -1}">
+                    <mass value=".5"/>
+                </xacro:if>
+                <xacro:if value="${front_hind == 1}">
+                    <mass value="${thigh_mass}"/>
+                    <!-- 1.152 -->
+                </xacro:if>
                 <inertia
                     ixx="${thigh_ixx}" ixy="${thigh_ixy*mirror}" ixz="${thigh_ixz}"
@@ -100,13 +106,13 @@
             </inertial>
         </link>
-        <joint name="${name}_calf_joint" type="revolute">
+        <joint name="${name}_lower_leg_joint" type="revolute">
             <origin rpy="0 0 0" xyz="0 0 ${-thigh_length}"/>
-            <parent link="${name}_thigh"/>
-            <child link="${name}_calf"/>
+            <parent link="${name}_upper_leg_link"/>
+            <child link="${name}_lower_leg_link"/>
             <axis xyz="0 1 0"/>
             <dynamics damping="${damping}" friction="${friction}"/>
             <limit effort="${calf_torque_max}" velocity="${calf_velocity_max}" lower="${calf_position_min}" upper="${calf_position_max}"/>
         </joint>
-        <link name="${name}_calf">
+        <link name="${name}_lower_leg_link">
             <visual>
                 <origin rpy="0 0 0" xyz="0 0 0"/>
@@ -131,10 +137,10 @@
             </inertial>
         </link>
-        <joint name="${name}_foot_fixed" type="fixed">0
+        <joint name="${name}_foot_joint" type="fixed">0
             <origin rpy="0 0 0" xyz="0 0 ${-(calf_length)}"/>
-            <parent link="${name}_calf"/>
-            <child link="${name}_foot"/>
-        </joint>
-        <link name="${name}_foot">
+            <parent link="${name}_lower_leg_link"/>
+            <child link="${name}_foot_link"/>
+        </joint>
+        <link name="${name}_foot_link">
             <visual>
                 <origin rpy="0 0 0" xyz="0 0 0"/>
@@ -158,4 +164,50 @@
             </inertial>
         </link>
+        <ros2_control name="${name}" type="system">
+            <hardware>
+                <plugin>gazebo_ros2_control/GazeboSystem</plugin>
+            </hardware>
+            <!-- ********************** FRONT RIGHT JOINTS *********************************  -->
+            <joint name="${name}_hip_joint">
+                <command_interface name="effort"/>
+                <state_interface name="position"/>
+                <state_interface name="velocity"/>
+            </joint>
+            <joint name="${name}_upper_leg_joint">
+                <command_interface name="effort"/>
+                <state_interface name="position"/>
+                <state_interface name="velocity"/>
+            </joint>
+            <joint name="${name}_lower_leg_joint">
+                <command_interface name="effort"/>
+                <state_interface name="position"/>
+                <state_interface name="velocity"/>
+            </joint>
+        </ros2_control>
+        <!-- RR leg -->
+        <gazebo reference="${name}_hip_link">
+            <mu1>0.2</mu1>
+            <mu2>0.2</mu2>
+        </gazebo>
+        <gazebo reference="${name}_upper_leg_link">
+            <mu1>0.2</mu1>
+            <mu2>0.2</mu2>
+            <self_collide>1</self_collide>
+            <kp  value="1000000.0"/>
+            <kd  value="1.0"/>
+        </gazebo>
+        <gazebo reference="${name}_lower_leg_link">
+            <mu1>0.2</mu1>
+            <mu2>0.2</mu2>
+            <self_collide>1</self_collide>
+        </gazebo>
+        <gazebo reference="${name}_foot_link">
+            <kp>10000000000.0</kp>
+            <kd>100.0</kd>
+            <mu1>0.8</mu1>
+            <mu2>0.8</mu2>
+            <minDepth>0.05</minDepth>
+            <material>Gazebo/FlatBlack</material>
+        </gazebo>
         <!-- <xacro:leg_transmission name="${name}"/> -->
     </xacro:macro>

File: go2_description/xacro/go2_robot.xacro (robot description, xacro)
@@ -4,5 +4,5 @@
     <xacro:include filename="$(find go2_description)/xacro/const.xacro"/>
     <xacro:include filename="$(find go2_description)/xacro/materials.xacro"/>
-    <xacro:include filename="$(find go2_description)/xacro/leg.xacro"/>
+    <xacro:include filename="$(find go2_description)/xacro/go2_leg.xacro"/>
     <!-- <xacro:include filename="/home/e-yantra/unitree_ws/install/go2_description/share/go2_description/xacro/const.xacro"/>
     <xacro:include filename="/home/e-yantra/unitree_ws/install/go2_description/share/go2_description/xacro/materials.xacro"/>
@@ -11,5 +11,5 @@
     <!-- find-pkg-share -->
     <!-- <xacro:include filename="$(find go2_description)/xacro/stairs.xacro"/> -->
-    <xacro:include filename="$(find go2_description)/xacro/gazebo.xacro"/>
+    <!-- <xacro:include filename="$(find go2_description)/urdf/gazebo.xacro"/> -->
     <!-- <xacro:include filename="$(find go2_gazebo)/launch/stairs.urdf.xacro"/> -->
     <!-- <xacro:stairs stairs="15" xpos="0" ypos="0" zpos="0" /> -->
@@ -20,10 +20,12 @@
     </xacro:if>  -->
     <!-- <link name="world"/>
+    <link name="map"/>
     <joint name="base_static_joint" type="fixed">
         <origin rpy="0 0 0" xyz="0 0 0"/>
         <parent link="world"/>
-        <child link="base"/>
+        <child link="map"/>
     </joint> -->
-    <link name="base">
+    <xacro:include filename="$(find go2_description)/xacro/accessories.urdf.xacro" />
+    <link name="base_link">
         <visual>
             <origin rpy="0 0 0" xyz="0 0 0"/>
@@ -35,5 +37,5 @@
     <joint name="floating_base" type="fixed">
         <origin rpy="0 0 0" xyz="0 0 0"/>
-        <parent link="base"/>
+        <parent link="base_link"/>
         <child link="trunk"/>
     </joint>
@@ -53,19 +55,25 @@
         </collision>
         <inertial>
-            <origin rpy="0 0 0" xyz="0.021112 0 -0.005366"/>
-            <!-- <origin rpy="0 0 0" xyz="${trunk_com_x} ${trunk_com_y} ${trunk_com_z}"/> -->
-            <mass value="6.921"/>
-            <!-- <mass value="${trunk_mass}"/> -->
-            <inertia
+            <!-- <origin rpy="0 0 0" xyz="0.021112 0 -0.005366"/> -->
+            <origin rpy="0 0 0" xyz="${trunk_com_x} ${trunk_com_y} ${trunk_com_z}"/>
+            <!-- <mass value="6.921"/> -->
+            <!-- <mass value="2"/> -->
+            <mass value="${trunk_mass}"/>
+            <!-- <inertia
                 ixx="0.02448" ixy="0.00012166" ixz="0.0014849"
                 iyy="0.098077" iyz="-3.12E-05"
-                izz="0.107"/>
-            <!-- <inertia
+                izz="0.107"/>   -->
+            <inertia
                 ixx="${trunk_ixx}" ixy="${trunk_ixy}" ixz="${trunk_ixz}"
                 iyy="${trunk_iyy}" iyz="${trunk_iyz}"
-                izz="${trunk_izz}"/>   -->
+                izz="${trunk_izz}"/>
         </inertial>
     </link>
-    <joint name="imu_joint" type="fixed">
+    <xacro:accessories
+        base_name="base_link"
+        base_length="0.3762"
+        base_height="0.114"
+    />
+    <!-- <joint name="imu_joint" type="fixed">
         <parent link="trunk"/>
         <child link="imu_link"/>
@@ -83,5 +91,5 @@
                 <box size="0.001 0.001 0.001"/>
             </geometry>
-            <!-- <material name="red"/> -->
+            <material name="red"/>
         </visual>
         <collision>
@@ -91,5 +99,5 @@
             </geometry>
         </collision>
-    </link>
+    </link> -->
     <!--
     <joint name="load_joint" type="fixed">
@@ -118,88 +126,26 @@
     </link>
 -->
-    <xacro:leg name="FR" mirror="-1" mirror_dae= "False" front_hind="1"  front_hind_dae="True"  />
-    <xacro:leg name="FL" mirror="1"  mirror_dae="True"   front_hind="1"  front_hind_dae="True"  />
-    <xacro:leg name="RR" mirror="-1" mirror_dae="False"  front_hind="-1" front_hind_dae="False" />
-    <xacro:leg name="RL" mirror="1"  mirror_dae="True"   front_hind="-1" front_hind_dae="False" />
-    <!-- <gazebo reference="FR_calf">
-        <material>Gazebo/Orange</material>
-        <kp>${kp}</kp>
-        <kd>${kd}</kd>
-        <mu1>${mu1}</mu1>
-        <mu2>${mu2}</mu2>
-        <maxVel>${max_vel}</maxVel>
-        <minDepth>${min_depth}</minDepth>
-    </gazebo> -->
-    <ros2_control name="GazeboSystem" type="system">
-        <hardware>
-            <plugin>gazebo_ros2_control/GazeboSystem</plugin>
-        </hardware>
-        <!-- ********************** FRONT RIGHT JOINTS *********************************  -->
-        <joint name="FR_hip_joint">
-            <command_interface name="effort"/>
-            <state_interface name="position"/>
-            <state_interface name="velocity"/>
-        </joint>
-        <joint name="FL_hip_joint">
-            <command_interface name="effort"/>
-            <state_interface name="position"/>
-            <state_interface name="velocity"/>
-        </joint>
-        <joint name="RR_hip_joint">
-            <command_interface name="effort"/>
-            <state_interface name="position"/>
-            <state_interface name="velocity"/>
-        </joint>
-        <joint name="RL_hip_joint">
-            <command_interface name="effort"/>
-            <state_interface name="position"/>
-            <state_interface name="velocity"/>
-        </joint>
-        <joint name="FR_thigh_joint">
-            <command_interface name="effort"/>
-            <state_interface name="position"/>
-            <state_interface name="velocity"/>
-        </joint>
-        <joint name="FL_thigh_joint">
-            <command_interface name="effort"/>
-            <state_interface name="position"/>
-            <state_interface name="velocity"/>
-        </joint>
-        <joint name="RR_thigh_joint">
-            <command_interface name="effort"/>
-            <state_interface name="position"/>
-            <state_interface name="velocity"/>
-        </joint>
-        <joint name="RL_thigh_joint">
-            <command_interface name="effort"/>
-            <state_interface name="position"/>
-            <state_interface name="velocity"/>
-        </joint>
-        <joint name="FR_calf_joint">
-            <command_interface name="effort"/>
-            <state_interface name="position"/>
-            <state_interface name="velocity"/>
-        </joint>
-        <joint name="FL_calf_joint">
-            <command_interface name="effort"/>
-            <state_interface name="position"/>
-            <state_interface name="velocity"/>
-        </joint>
-        <joint name="RR_calf_joint">
-            <command_interface name="effort"/>
-            <state_interface name="position"/>
-            <state_interface name="velocity"/>
-        </joint>
-        <joint name="RL_calf_joint">
-            <command_interface name="effort"/>
-            <state_interface name="position"/>
-            <state_interface name="velocity"/>
-        </joint>
-    </ros2_control>
+    <xacro:leg name="lf" mirror="1"  mirror_dae="True"   front_hind="1"  front_hind_dae="True"  />
+    <xacro:leg name="rf" mirror="-1" mirror_dae= "False" front_hind="1"  front_hind_dae="True"  />
+    <xacro:leg name="lh" mirror="1"  mirror_dae="True"   front_hind="-1" front_hind_dae="False" />
+    <xacro:leg name="rh" mirror="-1" mirror_dae="False"  front_hind="-1" front_hind_dae="False" />
+    <gazebo>
+      <plugin name="p3d_base_controller" filename="libgazebo_ros_p3d.so">
+        <ros>
+            <argument>odom:=odom/ground_truth</argument>
+        </ros>
+        <body_name>base_link</body_name>
+        <frame_name>world</frame_name>
+        <update_rate>10.0</update_rate>
+        <xyz_offset>0 0 0</xyz_offset>
+        <rpy_offset>0 0 0</rpy_offset>
+        <gaussian_noise>0.01</gaussian_noise>
+    </plugin>
+    </gazebo>
     <gazebo>
         <plugin filename="libgazebo_ros2_control.so" name="gazebo_ros2_control">
             <!-- <parameters>$(find-pkg-share go2_description)/config/go2_controlgdsf.yaml</parameters> -->
             <!-- <parameters>"${find go2_description}/config/go2_control.yaml"</parameters> -->
-            <parameters>$(find go2_description)/config/go2_control.yaml</parameters>
+            <parameters>$(find champ_gazebo)/config/go2_ros_control.yaml</parameters>
             <!-- <parameters>/home/e-yantra/unitree_ws/install/go2_description/share/go2_description/config/go2_control.yaml</parameters> -->
         </plugin>
