Commit message: minor cleanup and corrections

File: go2_description/xacro/hokuyo_utm30lx.urdf.xacro (robot description, xacro)
@@ -17,5 +17,5 @@
           <origin xyz="0 0 0" rpy="0 0 0" />
           <geometry>
-          <mesh filename="file://$(find champ_description)/meshes/hokuyo_utm_30lx$(optenv TEST_SELF_FILTER).dae"/>
+          <mesh filename="file://$(find go2_description)/meshes/hokuyo_utm_30lx$(optenv TEST_SELF_FILTER).dae"/>
         </geometry>
         </visual>
